Commit message: Need clean-up ASAP. Problem was the sponge's mesh, need to provide mesh with vertices uniformly distributed. New mesh worked! But need tuning and cleanup ASAP

File: urdf/biotac/shell_core/soft_body.urdf (robot description, URDF)
Before this commit: robot biotac, 3 links, 2 joints
Links:
- link arm: geometry collision box size=0.02 0.01 0.06

File: urdf/indenters/cylinder_long_7mm.urdf (robot description, URDF)
Before this commit: robot indenter, 2 links, 1 joints
Links:
- removed link world
Joints:
- removed joint world_to_indenter

File: urdf/indenters/plate_ycb_few.urdf (robot description, URDF)
Before this commit: robot indenter, 1 links, 0 joints
Links:
- link indenter: geometry collision mesh filename=../../meshes/target_objects/plate_ycb_few.obj; visual mesh filename=../../meshes/target_objects/plate_ycb_few.obj

Commit message: Added sampling points + normals. Now the gripper will approach the point through the its normal.

File: urdf/biotac/shell_core/soft_body.urdf (robot description, URDF)
Before this commit: robot biotac, 3 links, 2 joints
Links:
- link arm: geometry collision sphere radius=0.01

File: urdf/biotac/shell_core/sponge_template.urdf (robot description, URDF)
Before this commit: robot biotac, 3 links, 2 joints
Links:
- link arm: geometry collision sphere radius=0.01
