Commit message: Added data collection pipeline

File: urdf/targetobjects/bowl_shapenet.urdf (robot description, URDF)
Before this commit: robot indenter, 1 links, 0 joints
Links:
- link indenter: geometry collision mesh filename=../../meshes/target_objects/bowl_shapenet.obj; visual mesh filename=../../meshes/target_objects/bowl_shapenet.obj
